File: PCB/CodeBoard.kicad_pcb (KiCad board)
At the start: 2 copper layers, 371.7 x 98.1 mm, 164 parts, among them SW1 SW_Push, SW10 SW_Push, SW11 SW_Push, SW12 SW_Push, SW13 SW_Push, SW14 SW_Push, SW15 SW_Push, SW16 SW_Push, SW17 SW_Push, SW18 SW_Push, SW19 SW_Push, SW2 SW_Push, SW20 SW_Push, SW21 SW_Push, SW22 SW_Push, SW23 SW_Push, SW24 SW_Push, SW26 SW_Push, SW27 SW_Push, SW28 SW_Push, SW29 SW_Push, SW3 SW_Push, SW30 SW_Push, SW31 SW_Push, SW32 SW_Push, SW33 SW_Push, SW34 SW_Push, SW35 SW_Push, SW36 SW_Push, SW37 SW_Push, SW38 SW_Push, SW39 SW_Push, SW4 SW_Push, SW40 SW_Push, SW41 SW_Push, SW42 SW_Push, SW43 SW_Push, SW44 SW_Push, SW45 SW_Push, SW46 SW_Push, SW47 SW_Push, SW48 SW_Push, SW49 SW_Push, SW5 SW_Push, SW50 SW_Push, SW51 SW_Push, SW52 SW_Push, SW53 SW_Push, SW54 SW_Push, SW55 SW_Push, SW56 SW_Push, SW57 SW_Push, SW58 SW_Push, SW59 SW_Push, SW6 SW_Push, SW60 SW_Push, SW61 SW_Push, SW62 SW_Push, SW63 SW_Push, SW64 SW_Push, SW65 SW_Push, SW66 SW_Push, SW67 SW_Push, SW68 SW_Push, SW69 SW_Push, SW7 SW_Push, SW70 SW_Push, SW71 SW_Push, SW72 SW_Push, SW73 SW_Push, SW74 SW_Push, SW75 SW_Push, SW76 SW_Push, SW77 SW_Push, SW78 SW_Push, SW79 SW_Push, SW8 SW_Push, SW80 SW_Push, SW81 SW_Push, SW9 SW_Push

Commit message: Add files via upload
Connections:
- A1 pad 24: Col 0 -> Col 18
- A1 pad 25: Col 0 -> Row 0
- A1 pad 26: Col 0 -> Row 1
- A1 pad 27: Col 0 -> Row 2
- A1 pad 31: unconnected-(A1-GPIO26_ADC0-Pad31) -> Col 18
- D1 pad 1: Col 0 -> Row 0
- D10 pad 1: Col 0 -> Row 0
- D11 pad 1: Col 0 -> Row 0
- D12 pad 1: Col 0 -> Row 0
- D13 pad 1: Col 0 -> Row 1
- D14 pad 1: Col 0 -> Row 1
- D16 pad 1: Col 0 -> Row 0
- D17 pad 1: Col 0 -> Row 0
- D18 pad 1: Col 0 -> Row 0
- D19 pad 1: Col 0 -> Row 0
- D2 pad 1: Col 0 -> Row 0
- D20 pad 1: Col 0 -> Row 0
- D21 pad 1: Col 0 -> Row 1
- D22 pad 1: Col 0 -> Row 1
- D23 pad 1: Col 0 -> Row 1
- D24 pad 1: Col 0 -> Row 1
- D25 pad 1: Col 0 -> Row 1
- D26 pad 1: Col 0 -> Row 1
- D27 pad 1: Col 0 -> Row 1
- D28 pad 1: Col 0 -> Row 1
- D29 pad 1: Col 0 -> Row 1
- D3 pad 1: Col 0 -> Row 0
- D30 pad 1: Col 0 -> Row 1
- D31 pad 1: Col 0 -> Row 1
- D32 pad 1: Col 0 -> Row 1
- D33 pad 1: Col 0 -> Row 1
- D34 pad 1: Col 0 -> Row 1
- D35 pad 1: Col 0 -> Row 1
- D36 pad 1: Col 0 -> Row 2
- D37 pad 1: Col 0 -> Row 2
- D38 pad 1: Col 0 -> Row 2
- D39 pad 1: Col 0 -> Row 2
- D4 pad 1: Col 0 -> Row 0
- D40 pad 1: Col 0 -> Row 2
- D41 pad 1: Col 0 -> Row 2
- D42 pad 1: Col 0 -> Row 2
- D43 pad 1: Col 0 -> Row 2
- D44 pad 1: Col 0 -> Row 2
- D45 pad 1: Col 0 -> Row 2
- D46 pad 1: Col 0 -> Row 2
- D47 pad 1: Col 0 -> Row 2
- D48 pad 1: Col 0 -> Row 2
- D49 pad 1: Col 0 -> Row 2
- D5 pad 1: Col 0 -> Row 0
- D50 pad 1: Col 0 -> Row 2
- D51 pad 1: Col 0 -> Row 2
- D6 pad 1: Col 0 -> Row 0
- D69 pad 1: Col 0 -> Col 18
- D7 pad 1: Col 0 -> Row 0
- D70 pad 1: Col 0 -> Col 18
- D71 pad 1: Col 0 -> Col 18
- D72 pad 1: Col 0 -> Col 18
- D73 pad 1: Col 0 -> Col 18
- D74 pad 1: Col 0 -> Col 18
- D75 pad 1: Col 0 -> Col 18
- D76 pad 1: Col 0 -> Col 18
- D77 pad 1: Col 0 -> Col 18
- D78 pad 1: Col 0 -> Col 18
- D79 pad 1: Col 0 -> Col 18
- D8 pad 1: Col 0 -> Row 0
- D80 pad 1: Col 0 -> Col 18
- D81 pad 1: Col 0 -> Col 18
- D9 pad 1: Col 0 -> Row 0
- SW30 pad 1: Col 0 -> Col 18
- SW35 pad 1: Col 0 -> Col 18
Routing:
- net Col 18: track 0.00 -> 511.7 mm, vias 0 -> 4
- net Row 0: track 0.00 -> 414.4 mm, vias 0 -> 2
- net Row 1: track 0.00 -> 378.9 mm
- net Row 2: track 0.00 -> 330.6 mm
- net Col 0: track 1952.4 -> 1847.1 mm, vias 0 -> 1
- net Net-(D17-A): track 20.2 -> 26.2 mm
- net GND: track 95.2 -> 100.1 mm, vias 0 -> 2
- net Net-(D79-A): track 10.3 -> 13.9 mm
- net Net-(D70-A): track 18.6 -> 21.4 mm
- net Net-(D18-A): track 9.09 -> 11.9 mm
- net Net-(D55-A): track 10.4 -> 13.1 mm
- net Net-(D71-A): track 17.5 -> 20.1 mm
- net Net-(D58-A): track 24.4 -> 26.9 mm
- net Net-(D57-A): track 10.5 -> 12.9 mm
- net Net-(D81-A): track 10.2 -> 12.6 mm
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